Commit message: Added leg prototype, ros2 control, and fixed rviz

File: r2d2_robot_description/urdf/r2d2_body.urdf.xacro (robot description, xacro)
@@ -13,7 +13,5 @@
                     <sphere radius="1.5"/>
                 </geometry>
-                <material name="">
-                    <color rgba="1.0 0.0 0.0 1.0"/>
-                </material>
+                <material name="silver"/>
             </visual>
             <collision name='top_body_collision'>
@@ -36,7 +34,5 @@
                     <cylinder radius="1.5" length="2.0"/>
                 </geometry>
-                <material name="">
-                    <color rgba="1.0 0.0 0.0 1.0"/>
-                </material>
+                <material name="silver"/>
             </visual>
             <collision name='bottom_body_collision'>
@@ -47,8 +43,9 @@
             </collision>
         </link>
-        <joint name="body_joint" type="fixed">
+        <joint name="head_joint" type="revolute">
             <parent link="bottom_body"/>
             <child link="top_body"/>
             <origin xyz="0.0 0.0 1.0" rpy="0.0 0.0 0.0"/>
+            <limit lower="-1.0" upper="1.0" effort="0.0" velocity="1.0"/>
         </joint>
         <joint name="base_joint" type="fixed">

File: r2d2_robot_description/urdf/r2d2_leg.urdf.xacro (robot description, xacro)
@@ -1,6 +1,26 @@
 <?xml version="1.0"?>
 <robot xmlns:xacro="http://www.ros.org/wiki/xacro" name="r2d2">
-    <xacro:macro name="leg" params="wheel_1_name wheel_2_name body_joint_name">
-        <link name="top_leg">
+    <xacro:macro name="leg" params="side">
+        <link name="${side}_leg_top_link">
+            <inertial>
+                <origin xyz="0.0 0.0 0.0" rpy="0.0 0.0 0.0"/>
+                <mass value="5.0"/>
+                <inertia ixx="0.0" ixy="0.0" ixz="0.0" iyy="0.0" iyz="0.0" izz="0.0"/>
+            </inertial>
+            <visual name="${side}_leg_top_link_visual">
+                <origin xyz="0.0 0.0 0.0" rpy="1.5707 0.0 1.5707"/>
+                <geometry>
+                    <cylinder radius="0.3" length="0.5"/>
+                </geometry>
+                <material name="silver"/>
+            </visual>
+            <collision name="${side}_leg_top_link_collision">
+                <origin xyz="0.0 0.0 0.0" rpy="1.5707 0.0 1.5707"/>
+                <geometry>
+                    <cylinder radius="0.3" length="0.5"/>
+                </geometry>
+            </collision>
+        </link>
+        <link name="${side}_leg_middle_link">
             <inertial>
                 <origin xyz="0.0 0.0 0.0" rpy="0.0 0.0 0.0"/>
@@ -8,21 +28,35 @@
                 <inertia ixx="0.0" ixy="0.0" ixz="0.0" iyy="0.0" iyz="0.0" izz="0.0"/>
             </inertial>
-            <visual name="top_leg_visual">
+            <visual name="${side}_leg_middle_link_visual">
                 <origin xyz="0.0 0.0 0.0" rpy="0.0 0.0 0.0"/>
                 <geometry>
-                    <box size="1.0 1.0 2.0"/>
+                    <box size="0.3 1.0 2.0"/>
                 </geometry>
-                <material name="">
-                    <color rgba="1.0 0.0 0.0 1.0"/>
-                    <texture filename=""/>
-                </material>
+                <material name="silver"/>
             </visual>
-            <collision name="top_leg_collision">
+            <collision name="${side}_leg_middle_link_collision">
                 <origin xyz="0.0 0.0 0.0" rpy="0.0 0.0 0.0"/>
                 <geometry>
-                    <box size="1.0 1.0 2.0"/>
+                    <box size="0.3 1.0 2.0"/>
                 </geometry>
             </collision>
         </link>
+        <joint name="${side}_top_joint" type="fixed">
+            <xacro:if value='${side == "right"}'>
+                <origin xyz="2.0 0.0 0.5" rpy="0.0 0.0 0.0"/>
+            </xacro:if>
+            <xacro:unless value='${side == "right"}'>
+                <origin xyz="-2.0 0.0 0.5" rpy="0.0 0.0 0.0"/>
+            </xacro:unless>
+            <parent link="bottom_body"/>
+            <child link="${side}_leg_top_link"/>
+            <axis xyz="1.0 0.0 0.0"/>
+        </joint>
+        <joint name="${side}_middle_joint" type="fixed">
+            <origin xyz="0.0 0.0 -1.0" rpy="0.0 0.0 0.0"/>
+            <parent link="${side}_leg_top_link"/>
+            <child link="${side}_leg_middle_link"/>
+            <axis xyz="0.0 0.0 0.0"/>
+        </joint>
     </xacro:macro>
 </robot>

File: r2d2_robot_description/urdf/r2d2_rviz.urdf.xacro (robot description, xacro)
@@ -10,9 +10,6 @@
     </link>
     <xacro:body/>
-    <xacro:control hardware_flag='gazebo'/>
-    <gazebo>
-        <plugin filename="libgazebo_ros2_control.so" name="gazebo_ros2_control">
-            <parameters>$(find r2d2_robot_description)/config/ros2_controllers.yaml</parameters>
-        </plugin>
-    </gazebo>
+    <xacro:leg side='right'/>
+    <xacro:leg side='left'/>
+    <xacro:control hardware_flag='rviz'/>
 </robot>
