Commit message: Added inertia macros, wheels, and camera

File: r2d2_robot_description/urdf/general_macros.xacro (robot description, xacro)
@@ -1,3 +1,92 @@
 <?xml version="1.0"?>
 <robot xmlns:xacro="http://www.ros.org/wiki/xacro" name="r2d2">
+    <!-- Inertia tensors-->
+    <!-- Solid Sphere -->
+    <xacro:macro name="solid_sphere_inertia" params="m r">
+        <inertia
+            ixx="${(2*m*r*r)/5}"
+            ixy="0.0"
+            ixz="0.0"
+            iyy="${(2*m*r*r)/5}"
+            iyz="0.0"
+            izz="${(2*m*r*r)/5}"
+        />
+    </xacro:macro>
+    <!-- Hollow Sphere-->
+    <xacro:macro name="hollow_sphere_inertia" params="m r">
+        <inertia
+            ixx="${(2*m*r*r)/3}"
+            ixy="0.0"
+            ixz="0.0"
+            iyy="${(2*m*r*r)/3}"
+            iyz="0.0"
+            izz="${(2*m*r*r)/3}"
+        />
+    </xacro:macro>
+    <!-- Solid Ellipsoid-->
+    <xacro:macro name="solid_ellipsoid_inertia" params="m a b c">
+        <inertia
+            ixx="${(m*((b*b)+(c*c)))/5}"
+            ixy="0.0"
+            ixz="0.0"
+            iyy="${(m*((a*a)+(c*c)))/5}"
+            iyz="0.0"
+            izz="${(m*((b*b)+(a*a)))/5}"
+        />
+    </xacro:macro>
+    <!-- Right Circular Cone-->
+    <xacro:macro name="cone_inertia" params="r h m">
+        <inertia
+            ixx="${((3*m*h*h)/5)+((3*m*r*r)/20)}"
+            ixy="0.0"
+            ixz="0.0"
+            iyy="${((3*m*h*h)/5)+((3*m*r*r)/20)}"
+            iyz="0.0"
+            izz="${(3*m*r*r)/10}"
+        />
+    </xacro:macro>
+    <!-- Solid Cuboid-->
+    <xacro:macro name="solid_cuboid_inertia" params="m w h d">
+        <inertia
+            ixx="${(m*((h*h)+(d*d)))/12}"
+            ixy="0.0"
+            ixz="0.0"
+            iyy="${(m*((w*w)+(d*d)))/12}"
+            iyz="0.0"
+            izz="${(m*((w*w)+(h*h)))/12}"
+        />
+    </xacro:macro>
+    <!-- Slender Rod (y-axis, end) -->
+    <xacro:macro name="slender_rod_end_inertia" params="m l">
+        <inertia
+            ixx="${(m*l*l)/3}"
+            ixy="0.0"
+            ixz="0.0"
+            iyy="0.0"
+            iyz="0.0"
+            izz="${(m*l*l)/3}"
+        />
+    </xacro:macro>
+    <!-- Slender Rod (y-axis, center) -->
+    <xacro:macro name="slender_rod_center_inertia" params="m l">
+        <inertia
+            ixx="${(m*l*l)/12}"
+            ixy="0.0"
+            ixz="0.0"
+            iyy="0.0"
+            iyz="0.0"
+            izz="${(m*l*l)/12}"
+        />
+    </xacro:macro>
+    <!-- Solid Cyliner -->
+    <xacro:macro name="solid_cylinder_inertia" params="m r h">
+        <inertia
+            ixx="${(m*((3*r*r)+(h*h)))/12}"
+            ixy="0.0"
+            ixz="0.0"
+            iyy="${(m*((3*r*r)+(h*h)))/12}"
+            iyz="0.0"
+            izz="${(m*r*r)/2}"
+        />
+    </xacro:macro>
 </robot>

File: r2d2_robot_description/urdf/r2d2_body.urdf.xacro (robot description, xacro)
@@ -1,10 +1,18 @@
 <?xml version="1.0"?>
 <robot xmlns:xacro="http://www.ros.org/wiki/xacro" name="r2d2">
+    <!--
+        R2-D2 Main Body
+        Includes:
+        - Head
+        - Torso
+        - Camera
+    -->
     <xacro:macro name="body">
+        <!-- Head -->
         <link name="top_body">
             <inertial>
                 <origin xyz="0.0 0.0 0.0" rpy="0.0 0.0 0.0"/>
                 <mass value="20.0"/>
-                <inertia ixx="0.0" ixy="0.0" ixz="0.0" iyy="0.0" iyz="0.0" izz="0.0"/>
+                <xacro:solid_sphere_inertia m="20" r="1.5"/>
             </inertial>
             <visual name="top_body_visual">
@@ -22,4 +30,5 @@
             </collision>
         </link>
+        <!-- Torso -->
         <link name="bottom_body">
             <pose>0 0 0 0 0 0</pose>
@@ -27,10 +36,10 @@
                 <origin xyz="0.0 0.0 0.0" rpy="0.0 0.0 0.0"/>
                 <mass value="30.0"/>
-                <inertia ixx="0.0" ixy="0.0" ixz="0.0" iyy="0.0" iyz="0.0" izz="0.0"/>
+                <xacro:solid_cylinder_inertia m="30" h="3.0" r="1.5"/>
             </inertial>
             <visual name="bottom_body_visual">
                 <origin xyz="0.0 0.0 0.0" rpy="0.0 0.0 0.0"/>
                 <geometry>
-                    <cylinder radius="1.5" length="2.0"/>
+                    <cylinder radius="1.5" length="3.0"/>
                 </geometry>
                 <material name="silver"/>
@@ -39,5 +48,46 @@
                 <origin xyz="0.0 0.0 0.0" rpy="0.0 0.0 0.0"/>
                 <geometry>
-                    <cylinder radius="1.5" length="2.0"/>
+                    <cylinder radius="1.5" length="3.0"/>
+                </geometry>
+            </collision>
+        </link>
+        <!-- Camera -->
+        <link name="camera_housing">
+            <inertial>
+                <origin xyz="0.0 0.0 0.0" rpy="0.0 0.0 0.0"/>
+                <mass value="1.0"/>
+                <inertia ixx="0.0" ixy="0.0" ixz="0.0" iyy="0.0" iyz="0.0" izz="0.0"/>
+            </inertial>
+            <visual name="">
+                <origin xyz="0.0 0.0 0.0" rpy="0.0 0.0 0.0"/>
+                <geometry>
+                    <box size="0.5 0.4 0.5"/>
+                </geometry>
+                <material name="blue" />
+            </visual>
+            <collision>
+                <origin xyz="0.0 0.0 0.0" rpy="0.0 0.0 0.0"/>
+                <geometry>
+                    <box size="0.5 0.2 0.5"/>
+                </geometry>
+            </collision>
+        </link>
+        <link name="camera_optical_frame">
+            <inertial>
+                <origin xyz="0.0 0.0 0.0" rpy="0.0 0.0 0.0"/>
+                <mass value="1.0"/>
+                <inertia ixx="0.0" ixy="0.0" ixz="0.0" iyy="0.0" iyz="0.0" izz="0.0"/>
+            </inertial>
+            <visual name="">
+                <origin xyz="0.0 0.0 0.0" rpy="0.0 0.0 0.0"/>
+                <geometry>
+                    <sphere radius="0.15"/>
+                </geometry>
+                <material name="black"/>
+            </visual>
+            <collision>
+                <origin xyz="0.0 0.0 0.0" rpy="0.0 0.0 0.0"/>
+                <geometry>
+                    <sphere radius="0.15"/>
                 </geometry>
             </collision>
@@ -46,5 +96,5 @@
             <parent link="bottom_body"/>
             <child link="top_body"/>
-            <origin xyz="0.0 0.0 1.0" rpy="0.0 0.0 0.0"/>
+            <origin xyz="0.0 0.0 1.5" rpy="0.0 0.0 0.0"/>
             <limit lower="-1.0" upper="1.0" effort="0.0" velocity="1.0"/>
         </joint>
@@ -52,5 +102,17 @@
             <parent link="base_unit"/>
             <child link="bottom_body"/>
-            <origin xyz="0.0 0.0 1.5" rpy="0.0 0.0 0.0"/>
+            <origin xyz="0.0 0.0 2.5" rpy="0.0 0.0 0.0"/>
+        </joint>
+        <joint name="camera_housing_joint" type="fixed">
+            <origin xyz="0.0 1.25 0.6" rpy="0.0 0.0 0.0"/>
+            <parent link="top_body"/>
+            <child link="camera_housing"/>
+            <axis xyz="0.0 0.0 0.0"/>
+        </joint>
+        <joint name="camera_optical_joint" type="fixed">
+            <origin xyz="0.0 0.15 0.0" rpy="0.0 0.0 0.0"/>
+            <parent link="camera_housing"/>
+            <child link="camera_optical_frame"/>
+            <axis xyz="0.0 0.0 0.0"/>
         </joint>
     </xacro:macro>

File: r2d2_robot_description/urdf/r2d2_control.urdf.xacro (robot description, xacro)
@@ -21,4 +21,36 @@
                 <state_interface name='velocity'/>
             </joint>
+            <joint  name='right_front_wheel_joint'>
+                <command_interface name='velocity'>
+                    <param name='min'>-10</param>
+                    <param name='max'>10</param>
+                </command_interface>
+                <state_interface name='position'/>
+                <state_interface name='velocity'/>
+            </joint>
+            <joint  name='right_back_wheel_joint'>
+                <command_interface name='velocity'>
+                    <param name='min'>-10</param>
+                    <param name='max'>10</param>
+                </command_interface>
+                <state_interface name='position'/>
+                <state_interface name='velocity'/>
+            </joint>
+            <joint  name='left_front_wheel_joint'>
+                <command_interface name='velocity'>
+                    <param name='min'>-10</param>
+                    <param name='max'>10</param>
+                </command_interface>
+                <state_interface name='position'/>
+                <state_interface name='velocity'/>
+            </joint>
+            <joint  name='left_back_wheel_joint'>
+                <command_interface name='velocity'>
+                    <param name='min'>-10</param>
+                    <param name='max'>10</param>
+                </command_interface>
+                <state_interface name='position'/>
+                <state_interface name='velocity'/>
+            </joint>
         </ros2_control>
     </xacro:macro>

File: r2d2_robot_description/urdf/r2d2_leg.urdf.xacro (robot description, xacro)
@@ -6,5 +6,5 @@
                 <origin xyz="0.0 0.0 0.0" rpy="0.0 0.0 0.0"/>
                 <mass value="5.0"/>
-                <inertia ixx="0.0" ixy="0.0" ixz="0.0" iyy="0.0" iyz="0.0" izz="0.0"/>
+                <xacro:solid_cylinder_inertia m="5" h="0.5" r="0.3"/>
             </inertial>
             <visual name="${side}_leg_top_link_visual">
@@ -26,10 +26,10 @@
                 <origin xyz="0.0 0.0 0.0" rpy="0.0 0.0 0.0"/>
                 <mass value="10.0"/>
-                <inertia ixx="0.0" ixy="0.0" ixz="0.0" iyy="0.0" iyz="0.0" izz="0.0"/>
+                <xacro:solid_cuboid_inertia m="10" h="2.5" d="0.3" w="1.0"/>
             </inertial>
             <visual name="${side}_leg_middle_link_visual">
                 <origin xyz="0.0 0.0 0.0" rpy="0.0 0.0 0.0"/>
                 <geometry>
-                    <box size="0.3 1.0 2.0"/>
+                    <box size="0.3 1.0 2.5"/>
                 </geometry>
                 <material name="silver"/>
@@ -38,5 +38,65 @@
                 <origin xyz="0.0 0.0 0.0" rpy="0.0 0.0 0.0"/>
                 <geometry>
-                    <box size="0.3 1.0 2.0"/>
+                    <box size="0.3 1.0 2.5"/>
+                </geometry>
+            </collision>
+        </link>
+        <link name="${side}_leg_foot_link">
+            <inertial>
+                <origin xyz="0.0 0.0 0.0" rpy="0.0 0.0 0.0"/>
+                <mass value="5.0"/>
+                <xacro:solid_cuboid_inertia m="5" h="0.5" d="1" w="1"/>
+            </inertial>
+            <visual name="">
+                <origin xyz="0.0 0.0 0.0" rpy="0.0 0.0 0.0"/>
+                <geometry>
+                    <box size="1.0 1.0 0.5"/>
+                </geometry>
+                <material name='silver'/>
+            </visual>
+            <collision>
+                <origin xyz="0.0 0.0 0.0" rpy="0.0 0.0 0.0"/>
+                <geometry>
+                    <box size="1.0 1.0 0.5"/>
+                </geometry>
+            </collision>
+        </link>
+        <link name="${side}_front_wheel_link">
+            <inertial>
+                <origin xyz="0.0 0.0 0.0" rpy="0.0 0.0 0.0"/>
+                <mass value="1.0"/>
+                <xacro:solid_cylinder_inertia m="1.0" h="0.75" r="0.25"/>
+            </inertial>
+            <visual name="">
+                <origin xyz="0.0 0.0 0.0" rpy="1.5707 0.0 1.5707"/>
+                <geometry>
+                    <cylinder radius="0.25" length="0.75"/>
+                </geometry>
+                <material name="silver"/>
+            </visual>
+            <collision>
+                <origin xyz="0.0 0.0 0.0" rpy="1.5707 0.0 1.5707"/>
+                <geometry>
+                    <cylinder radius="0.25" length="0.75"/>
+                </geometry>
+            </collision>
+        </link>
+        <link name="${side}_back_wheel_link">
+            <inertial>
+                <origin xyz="0.0 0.0 0.0" rpy="0.0 0.0 0.0"/>
+                <mass value="1.0"/>
+                <xacro:solid_cylinder_inertia m="1.0" h="0.75" r="0.25"/>
+            </inertial>
+            <visual name="">
+                <origin xyz="0.0 0.0 0.0" rpy="1.5707 0.0 1.5707"/>
+                <geometry>
+                    <cylinder radius="0.25" length="0.75"/>
+                </geometry>
+                <material name="silver"/>
+            </visual>
+            <collision>
+                <origin xyz="0.0 0.0 0.0" rpy="1.5707 0.0 1.5707"/>
+                <geometry>
+                    <cylinder radius="0.25" length="0.75"/>
                 </geometry>
             </collision>
@@ -44,8 +104,8 @@
         <joint name="${side}_top_joint" type="fixed">
             <xacro:if value='${side == "right"}'>
-                <origin xyz="2.0 0.0 0.5" rpy="0.0 0.0 0.0"/>
+                <origin xyz="1.75 0.0 0.75" rpy="0.0 0.0 0.0"/>
             </xacro:if>
             <xacro:unless value='${side == "right"}'>
-                <origin xyz="-2.0 0.0 0.5" rpy="0.0 0.0 0.0"/>
+                <origin xyz="-1.75 0.0 0.75" rpy="0.0 0.0 0.0"/>
             </xacro:unless>
             <parent link="bottom_body"/>
@@ -54,9 +114,27 @@
         </joint>
         <joint name="${side}_middle_joint" type="fixed">
-            <origin xyz="0.0 0.0 -1.0" rpy="0.0 0.0 0.0"/>
+            <origin xyz="0.0 0.0 -1.25" rpy="0.0 0.0 0.0"/>
             <parent link="${side}_leg_top_link"/>
             <child link="${side}_leg_middle_link"/>
             <axis xyz="0.0 0.0 0.0"/>
         </joint>
+        <joint name="${side}_foot_joint" type="fixed">
+            <origin xyz="0.0 0.0 -1.5" rpy="0.0 0.0 0.0"/>
+            <parent link="${side}_leg_middle_link"/>
+            <child link="${side}_leg_foot_link"/>
+            <axis xyz="0.0 0.0 0.0"/>
+        </joint>
+        <joint name="${side}_front_wheel_joint" type="continuous">
+            <origin xyz="0.0 0.25 -0.1" rpy="0.0 0.0 0.0"/>
+            <parent link="${side}_leg_foot_link"/>
+            <child link="${side}_front_wheel_link"/>
+            <axis xyz="0.0 1 0.0"/>
+        </joint>
+        <joint name="${side}_back_wheel_joint" type="continuous">
+            <origin xyz="0.0 -0.25 -0.1" rpy="0.0 0.0 0.0"/>
+            <parent link="${side}_leg_foot_link"/>
+            <child link="${side}_back_wheel_link"/>
+            <axis xyz="0.0 1 0.0"/>
+        </joint>
     </xacro:macro>
 </robot>
