Commit message: Added gazebo launch and drivers for easy control

File: r2d2_robot_description/urdf/r2d2.urdf.xacro (robot description, xacro)
@@ -4,4 +4,5 @@
     <xacro:include filename="$(find r2d2_robot_description)/urdf/r2d2_body.urdf.xacro"/>
     <xacro:include filename="$(find r2d2_robot_description)/urdf/r2d2_control.urdf.xacro"/>
+    <xacro:include filename="$(find r2d2_robot_description)/urdf/r2d2.gazebo.xacro"/>
     <xacro:include filename="$(find r2d2_robot_description)/urdf/general_macros.xacro"/>
     <xacro:include filename="$(find r2d2_robot_description)/urdf/materials.xacro"/>
@@ -10,4 +11,7 @@
     </link>
     <xacro:body/>
+    <xacro:leg side='right'/>
+    <xacro:leg side='left'/>
+    <xacro:gazebo_tags />
     <xacro:control hardware_flag='gazebo'/>
     <gazebo>

File: r2d2_robot_description/urdf/r2d2_body.urdf.xacro (robot description, xacro)
@@ -97,4 +97,5 @@
             <child link="top_body"/>
             <origin xyz="0.0 0.0 1.5" rpy="0.0 0.0 0.0"/>
+            <axis xyz="0.0 0.0 1.0"/>
             <limit lower="-1.0" upper="1.0" effort="0.0" velocity="1.0"/>
         </joint>

File: r2d2_robot_description/urdf/r2d2_leg.urdf.xacro (robot description, xacro)
@@ -129,5 +129,5 @@
             <parent link="${side}_leg_foot_link"/>
             <child link="${side}_front_wheel_link"/>
-            <axis xyz="0.0 1 0.0"/>
+            <axis xyz="1 0.0 0.0"/>
         </joint>
         <joint name="${side}_back_wheel_joint" type="continuous">
@@ -135,5 +135,5 @@
             <parent link="${side}_leg_foot_link"/>
             <child link="${side}_back_wheel_link"/>
-            <axis xyz="0.0 1 0.0"/>
+            <axis xyz="1 0.0 0.0"/>
         </joint>
     </xacro:macro>
